File: G5 préamp/PCB_main/pcb_main.kicad_pcb (KiCad board)
At the start: 2 copper layers, 165 x 58 mm, 48 parts, among them J1 PSU_TUBE, J2 PCB_TUBE, J3 PSU_AMP, J4 AMP, J5 PSU_SIMCAB, J6 SIMCAB, J8 LEVEL 3-2, SW1 Boost, SW2 SIMCAB

Commit message: Add files via upload
Parts:
- removed REF**: PG5_Logo_15mm_SilkScreen, Symbol:PG5_Logo_15mm_SilkScreen
Connections:
- Ouput1 pad S: GNDS -> Net-(GND1-Pad1)
Routing:
- net Net-(GND1-Pad1): track 23.1 -> 67.8 mm
- net GNDS: track 595.3 -> 580.3 mm
