File: G5_preamp/RC1/PCB_main_alt/pcb_main.kicad_pcb (KiCad board)
At the start: 2 copper layers, 165 x 58 mm, 57 parts, among them J1 PSU_TUBE, J2 PCB_TUBE, J3 PSU_AMP, J4 AMP, J5 PSU_SIMCAB, J6 SIMCAB, J7 3PDT, J8 LEVEL 3-2, Q1 MPS751, Q2 IRF740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

Commit message: Validation RC1
Commande PCB
Parts:
- added REF**: PG5_Logo_15mm_SilkScreen, Symbol:PG5_Logo_15mm_SilkScreen, F.Cu at (200.8, 133.8)
- renumbered Ouput2 to HP, Input1 to Input, Ouput1 to Ouput
