File: G5_preamp/RC2/PCB_main/pcb_main.kicad_pcb (KiCad board)
At the start: 2 copper layers, 165 x 58 mm, 58 parts, among them J1 PSU_TUBE, J2 PCB_TUBE, J3 PSU_AMP, J4 AMP, J5 PSU_SIMCAB, J6 SIMCAB, J7 3PDT, J8 LEVEL 3-2, Q1 MPS751, Q2 IRF740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

Commit message: GND lift arrangement
GND lift arrangement
Parts:
- GND1: footprint Connector_Wire:SolderWirePad_1x02_P7.62mm_Drill2mm -> Connector_Wire:SolderWirePad_1x03_P3.175mm_Drill1mm
Connections:
- GND1 pad 2: GNDS -> Net-(GND1-Pad2)
- OT1 pad 1: Net-(GND1-Pad1) -> Net-(GND1-Pad2)
- R18 pad 2: Net-(GND1-Pad1) -> Net-(GND1-Pad2)
- R20 pad 2: Net-(GND1-Pad1) -> Net-(GND1-Pad2)
- XLR1 pad 1: GNDS -> Net-(GND1-Pad1)
Routing:
- net Net-(GND1-Pad2): track 0.00 -> 28.3 mm
- net GNDS: track 367.9 -> 347.3 mm
- net Net-(GND1-Pad1): track 67.6 -> 69.7 mm
