File: G5_preamp/RC5/PCB_tube/pcb_tube.kicad_pcb (KiCad board)
At the start: 2 copper layers, 96 x 47 mm, 33 parts, among them J1 PSU_TUBE, J2 PCB_TUBE, J3 OT, J9 Voltage_Heater, U1 PG5_Logo

Commit message: Update pcb_tube.kicad_pcb
Parts:
- moved H1 0.40 mm to (48.6, 94.3)
- moved J1 0.40 mm to (114.4, 84.3)
- moved J2 0.40 mm to (83.5, 84.3)
- moved JP1 0.38 mm to (52.3, 98.3)
Routing:
- net /K_V1B: track 43.9 -> 44.8 mm
- net /NFB: track 51.6 -> 52.4 mm
- net /HT2: track 9.78 -> 9.22 mm
Other:
- board size 96 x 47 mm -> 96 x 46.6 mm

Commit message: update pcb_main tracks
Changed lines of the file:
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@@
     (descr "simple 3-pin terminal block, pitch 5.08mm, revamped version of bornier3")
     (tags "terminal block bornier3")
-    (fp_text reference J3 (at -2.06 4.93 180) (layer F.SilkS)
+    (fp_text reference J3 (at 12.06 4.8 180) (layer F.SilkS)
       (effects (font (size 1 1) (thickness 0.15)))
     )
@@
     (arrow2b (pts (xy 30 100.9) (xy 31.126504 100.313579)))
   )
-  (gr_text or (at 52.8 54) (layer F.SilkS)
+  (gr_text or (at 52.57 54.06) (layer F.SilkS)
     (effects (font (size 1 1) (thickness 0.1)))
   )
@@
     (effects (font (size 1 1) (thickness 0.15)))
   )
-  (gr_text "G5 Preamp\nwith Pistorsion \nSystem" (at 106.68 82.33) (layer F.SilkS)
+  (gr_text "G5 Preamp\nwith Pistorsion \nSystem" (at 106.22 93.83) (layer F.SilkS)
     (effects (font (size 1 1) (thickness 0.15)))
   )
